File: CoquiKeyboard.kicad_sch (KiCad schematic)
At the start: 155 parts, among them J1 TYPE-C-31-M12_13, SW1 MXSwitch, SW10 MXSwitch, SW11 MXSwitch, SW12 MXSwitch, SW13 MXSwitch, SW14 MXSwitch, SW15 MXSwitch, SW16 MXSwitch, SW17 MXSwitch, SW18 MXSwitch, SW19 MXSwitch, SW2 MXSwitch, SW20 MXSwitch, SW21 MXSwitch, SW22 MXSwitch, SW23 MXSwitch, SW24 MXSwitch, SW25 MXSwitch, SW26 MXSwitch, SW27 MXSwitch, SW28 MXSwitch, SW29 MXSwitch, SW3 MXSwitch, SW30 MXSwitch, SW31 MXSwitch, SW32 MXSwitch, SW33 MXSwitch, SW34 MXSwitch, SW35 MXSwitch, SW36 MXSwitch, SW37 MXSwitch, SW38 MXSwitch, SW39 MXSwitch, SW4 MXSwitch, SW40 MXSwitch, SW41 MXSwitch, SW42 MXSwitch, SW43 MXSwitch, SW44 MXSwitch, SW45 MXSwitch, SW46 MXSwitch, SW47 MXSwitch, SW48 MXSwitch, SW49 MXSwitch, SW5 MXSwitch, SW50 MXSwitch, SW51 MXSwitch, SW52 MXSwitch, SW53 MXSwitch, SW54 MXSwitch, SW55 MXSwitch, SW56 MXSwitch, SW57 MXSwitch, SW58 MXSwitch, SW6 MXSwitch, SW7 MXSwitch, SW8 MXSwitch, SW9 MXSwitch, U1 STM32F303-LQFP48, U2 USBLC6-2SC6, U3 MCP1700-3302E_SOT23, Y1 8MHz

Commit message: finalized
Parts:
- removed H1, H6: MountingHole, MountingHole:MountingHole_2.5mm_Pad, symbol Mechanical:MountingHole
- removed H4: MountingHole, MountingHole:MountingHole_2.5mm_Pad, symbol Mechanical:MountingHole_Pad
- removed RF1: 100k, acheron_Components:R_SMD_1206, symbol Device:R
- added H4: MountingHole, MountingHole:MountingHole_2.5mm_Pad, symbol Mechanical:MountingHole
- added H6: MountingHole, MountingHole:MountingHole_2.5mm_Pad, symbol Mechanical:MountingHole_Pad
- DF1, DS1: footprint Diode_SMD:D_SOD-123 -> acheron_Components:D_SOD-123
- F1: footprint Fuse:Fuse_1206_3216Metric_Pad1.42x1.75mm_HandSolder -> acheron_Components:Fuse_1812_4532
- RDN1, RDP1, RDPUp1: footprint Resistor_SMD:R_1206_3216Metric_Pad1.30x1.75mm_HandSolder -> acheron_Components:R_SMD_1206
Connections:
- net Col1 is gone; now on net COL1: SW1.1 (Col), SW17.1 (Col), SW32.1 (Col), SW47.1 (Col)
- net Col10 is gone; now on net COL10: SW10.1 (Col), SW26.1 (Col), SW40.1 (Col)
- net Col11 is gone; now on net COL11: SW11.1 (Col), SW27.1 (Col), SW41.1 (Col), SW53.1 (Col)
- net Col12 is gone; now on net COL12: SW12.1 (Col), SW28.1 (Col), SW42.1 (Col), SW54.1 (Col)
- net Col13 is gone; now on net COL13: SW13.1 (Col), SW43.1 (Col), SW55.1 (Col)
- net Col15 is gone; now on net COL15: SW15.1 (Col), SW30.1 (Col), SW45.1 (Col), SW57.1 (Col)
- net Col16 is gone; now on net COL16: SW16.1 (Col), SW31.1 (Col), SW46.1 (Col), SW58.1 (Col)
- net Col2 is gone; now on net COL2: SW18.1 (Col), SW2.1 (Col), SW48.1 (Col)
- net Col3 is gone; now on net COL3: SW19.1 (Col), SW3.1 (Col), SW33.1 (Col), SW49.1 (Col)
- net Col4 is gone; now on net COL4: SW20.1 (Col), SW34.1 (Col), SW4.1 (Col), SW50.1 (Col)
- net Col5 is gone; now on net COL5: SW21.1 (Col), SW35.1 (Col), SW5.1 (Col)
- net Col6 is gone; now on net COL6: SW22.1 (Col), SW36.1 (Col), SW51.1 (Col), SW6.1 (Col)
- net Col7 is gone; now on net COL7: SW23.1 (Col), SW37.1 (Col), SW7.1 (Col)
- net Col8 is gone; now on net COL8: SW24.1 (Col), SW38.1 (Col), SW8.1 (Col)
- net Col9 is gone; now on net COL9: SW25.1 (Col), SW39.1 (Col), SW52.1 (Col), SW9.1 (Col)
- net Row1 is gone; now on net ROW1: D1.1 (K), D10.1 (K), D11.1 (K), D12.1 (K), D13.1 (K), D14.1 (K), D15.1 (K), D16.1 (K), D2.1 (K), D3.1 (K), D4.1 (K), D5.1 (K), D6.1 (K), D7.1 (K), D8.1 (K), D9.1 (K)
- net Row2 is gone; now on net ROW2: D17.1 (K), D18.1 (K), D19.1 (K), D20.1 (K), D21.1 (K), D22.1 (K), D23.1 (K), D24.1 (K), D25.1 (K), D26.1 (K), D27.1 (K), D28.1 (K), D29.1 (K), D30.1 (K), D31.1 (K)
- net Row3 is gone; now on net ROW3: D32.1 (K), D33.1 (K), D34.1 (K), D35.1 (K), D36.1 (K), D37.1 (K), D38.1 (K), D39.1 (K), D40.1 (K), D41.1 (K), D42.1 (K), D43.1 (K), D44.1 (K), D45.1 (K), D46.1 (K)
- net Row4 is gone; now on net ROW4: D47.1 (K), D48.1 (K), D49.1 (K), D50.1 (K), D51.1 (K), D52.1 (K), D53.1 (K), D54.1 (K), D55.1 (K), D56.1 (K), D57.1 (K), D58.1 (K)
- net COL1: now also U1.38 (PA15); no longer U1.22 (PB11)
- net COL11: now also U1.2 (PC13); no longer U1.12 (PA2)
- net COL12: now also U1.3 (PC14/OSC32_IN); no longer U1.11 (PA1)
- net COL13: now also U1.4 (PC15/OSC32_OUT); no longer U1.10 (PA0)
- net COL15: now also U1.17 (PA7); no longer U1.40 (PB4)
- net COL16: now also U1.16 (PA6); no longer U1.41 (PB5)
- net COL2: now also U1.39 (PB3); no longer U1.21 (PB10)
- net COL3: now also U1.40 (PB4); no longer U1.20 (PB2)
- net COL4: now also U1.41 (PB5); no longer U1.19 (PB1)
- net COL5: now also U1.42 (PB6); no longer U1.18 (PB0)
- net COL6: now also U1.43 (PB7); no longer U1.17 (PA7)
- net COL7: now also U1.45 (PB8); no longer U1.16 (PA6)
- net COL8: now also U1.46 (PB9); no longer U1.15 (PA5)
- net ROW1: now also U1.29 (PA8); no longer U1.38 (PA15)
- net ROW2: now also U1.21 (PB10); no longer U1.39 (PB3)
- net ROW3: now also U1.18 (PB0); no longer U1.42 (PB6)
- net ROW4: now also U1.20 (PB2); no longer U1.43 (PB7)
- net Col14 renamed COL14
- new net CASE: H6.1
Other:
- note added: "Switch matrix"

Commit message: close traces
Parts:
- CB1, CB2, CB3, CF1, CRO1: LCSC part number (none) -> C111492; Package (none) -> 0805
- CB4: LCSC part number (none) -> C141772; Package (none) -> 0805
- CB5: LCSC part number (none) -> C58456; Package (none) -> 0805
- CB6, CRST1, CSH1, CUSB1: LCSC part number (none) -> C37818; Package (none) -> 0805
- CRST2: LCSC part number (none) -> C15850; Package (none) -> 0805
- CX1, CX2: LCSC part number (none) -> C1804; Package (none) -> 0805
- D1, D10, D11, D12, D13, D14, D15, D16, D17, D18, D19, D2, D20, D21, D22, D23, D24, D25, D26, D27, D28, D29, D3, D30, D31, D32, D33, D34, D35, D36, D37, D38, D39, D4, D40, D41, D42, D43, D44, D45, D46, D47, D48, D49, D5, D50, D51, D52, D53, D54, D55, D56, D57, D58, D6, D7, D8, D9, DRST1: value 1N4148 -> 1N4148W; LCSC part number (none) -> C181134; Package (none) -> SOD-123
- DF1: LCSC part number (none) -> C114257; Package (none) -> SOD-123
- DS1: value 1N4007 -> 1N4007W; LCSC part number (none) -> C108803; Package (none) -> SOD-123
- F1: value 1A trip polyfuse -> 1A; footprint acheron_Components:Fuse_1812_4532 -> Fuse:Fuse_0805_2012Metric_Pad1.15x1.40mm_HandSolder; LCSC part number (none) -> C20979; Package (none) -> 0805
- J1: LCSC part number (none) -> C165948
- QRST1: LCSC part number (none) -> C111724; Package (none) -> SOT-23
- RCC1, RCC2: LCSC part number (none) -> C352054; Package (none) -> 1206
- RDN1, RDP1: LCSC part number (none) -> C17958; Package (none) -> 1206
- RDPUp1: LCSC part number (none) -> C212489; Package (none) -> 1206
- RRST1: LCSC part number (none) -> C212480; Package (none) -> 1206
- RSH1: LCSC part number (none) -> C308486; Package (none) -> 1206
- SRST1: LCSC part number (none) -> C92584; Package (none) -> SPST-NO
- U1: LCSC part number (none) -> C81523
- U2: LCSC part number (none) -> C7519; Package (none) -> SOT-23-6
- U3: LCSC part number (none) -> C39051; Package (none) -> SOT-23
- Y1: LCSC part number (none) -> C251594; Package (none) -> 5032 4Pin
Connections:
- net COL10: now also U1.3 (PC14/OSC32_IN); no longer U1.13 (PA3)
- net COL11: now also U1.4 (PC15/OSC32_OUT); no longer U1.2 (PC13)
- net COL12: now also U1.10 (PA0); no longer U1.3 (PC14/OSC32_IN)
- net COL13: now also U1.11 (PA1); no longer U1.4 (PC15/OSC32_OUT)
- net COL9: now also U1.2 (PC13); no longer U1.14 (PA4)
